File: HD-AK4316.kicad_sch (KiCad schematic)
At the start: 17 parts, among them CN1 HY-2-THRU, CN2 HY-2-THRU, U1 AE-LTC4316, U2 MIC5219-3.3YM5, U3 LP2950L-33-T92-K

Commit message: update: U2: partsnumber
Parts:
- U2: value MIC5219-3.3YM5 -> TPS74033
Changed lines of the file:
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@@
       (effects (font (size 1.27 1.27)))
     )
-    (property "Value" "MIC5219-3.3YM5" (at 71.12 161.29 0)
+    (property "Value" "TPS74033" (at 71.12 161.29 0)
       (effects (font (size 1.27 1.27)))
     )
